File: PCB/pulse oximeter.kicad_pcb (KiCad board)
At the start: 2 copper layers, 51.6 x 22.5 mm, 40 parts, among them J1 USB_C_Receptacle_USB2.0_14P, J2 Conn_01x04_Socket, J3 Conn_01x02_Socket, Q1 FS8205A, SW1 SW_Push, SW2 RESET, U1 ATMEGA328P-AU, U2 AP2112K-3.3TRG1, U3 DW01A, U4 MAX30102EFD_, U5 MCP73831-2-OT, U6 CH340C, Y1 8MHz

Commit message: Organized files
Parts:
- C1, C2: footprint Capacitor_SMD:C_0603_1608Metric -> Resistor_SMD:R_0201_0603Metric
- moved C2 4.35 mm to (135.0, 107.5)
- moved C1 3.26 mm to (136.7, 107.5)
Connections:
- Q1 pad 3: unconnected-(Q1-Pad3) -> BGND
Routing:
- net BGND: track 7.15 -> 48.3 mm, vias 1 -> 2
- net GND: track 136.9 -> 141.2 mm
- net BVCC: track 37.9 -> 34.0 mm
- net Net-(U1-PB7): track 16.3 -> 13.8 mm
- net Net-(U3-OC): track 5.20 -> 7.57 mm
- net Net-(U3-OD): track 14.3 -> 13.2 mm
- net Net-(U1-PB6): track 15.4 -> 16.2 mm, vias 4 -> 2
Other:
- board size 51.6 x 22.5 mm -> 51.6 x 22.6 mm
