File: PCB/pulse oximeter.kicad_sch (KiCad schematic)
At the start: 36 parts, among them J1 USB_C_Receptacle_USB2.0_14P, J2 Conn_01x04_Socket, J3 Conn_01x02_Socket, Q1 FS8205A, SW1 SW_Push, SW2 RESET, U1 ATMEGA328P-AU, U2 AP2112K-3.3TRG1, U3 DW01A, U4 MAX30102EFD_, U5 MCP73831-2-OT, U6 CH340C, Y1 8MHz

Commit message: Organized files
Parts:
- C1, C10, C2, C9: MPN (none) -> CL10A475KQ8NNNC
- C11, C3, C4, C5, C6, C7: MPN (none) -> CL10B104KB8NNNC
- C8: MPN (none) -> C0603C105K9RACAUTO
- D1: MPN (none) -> CMD17-21VRD/TR8
- J1: MPN (none) -> 12402012E212A
- Q1: MPN (none) -> FS8205A
- R1, R2: MPN (none) -> FRC0603F5101TS
- R10, R6: MPN (none) -> FRC0603F1001TS
- R11: MPN (none) -> 0603WAF2001T5E
- R3, R4: MPN (none) -> RC0603FR-0710KL
- R5: MPN (none) -> 0603WAF4700T5E
- R7: MPN (none) -> Y4021100R000B9W
- R8, R9: MPN (none) -> RC0603FR-074K7L
- SW1, SW2: MPN (none) -> KMR641NG ULC LFS
- U1: MPN (none) -> ATMEGA328P-AU
- U2: MPN (none) -> AP2112K-3.3TRG1
- U3: MPN (none) -> DW01A
- U4: MPN (none) -> MAX30102EFD+
- U5: MPN (none) -> MCP73831T-2ACI/OT
- U6: MPN (none) -> CH340C
- Y1: MPN (none) -> X32258MOB4SI
